File: SLT-5ns_AOI11-Family/361412_AOI11B/361412_AOI11B.kicad_sch (KiCad schematic)
At the start: 20 parts, among them T1 T_DB, T2 T_DA

Commit message: Updated schematics
Other:
- note removed: "B"
- note removed: "C"
- note removed: "E"
- note removed: "Transistor Die Layout (top view)"
Changed lines of the file:
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@@
     (stroke (width 0) (type default) (color 0 0 0 0))
-  )
-  (polyline (pts (xy 252.73 29.21) (xy 252.73 40.64))
-    (stroke (width 0) (type solid) (color 0 0 0 0))
   )
   (wire (pts (xy 53.34 72.39) (xy 60.96 72.39))
     (stroke (width 0) (type default) (color 0 0 0 0))
-  )
-  (polyline (pts (xy 264.16 40.64) (xy 252.73 40.64))
-    (stroke (width 0) (type solid) (color 0 0 0 0))
   )
   (wire (pts (xy 138.43 115.57) (xy 147.32 115.57))
@@
   (wire (pts (xy 78.74 58.42) (xy 68.58 58.42))
     (stroke (width 0) (type default) (color 0 0 0 0))
-  )
-  (polyline (pts (xy 252.73 29.21) (xy 264.16 29.21))
-    (stroke (width 0) (type solid) (color 0 0 0 0))
   )
   (wire (pts (xy 132.08 78.74) (xy 120.65 78.74))
@@
   (wire (pts (xy 152.4 143.51) (xy 152.4 139.7))
     (stroke (width 0) (type default) (color 0 0 0 0))
-  )
-  (polyline (pts (xy 264.16 29.21) (xy 264.16 40.64))
-    (stroke (width 0) (type solid) (color 0 0 0 0))
   )
   (wire (pts (xy 139.7 66.04) (xy 152.4 66.04))
@@
     (effects (font (size 1.27 1.27)) (justify left bottom))
   )
-  (text "C" (at 257.81 39.37 0)
-    (effects (font (size 1.27 1.27)) (justify left bottom))
-  )
   (text "AND Extend" (at 59.69 147.32 0)
     (effects (font (size 1.27 1.27)) (justify left bottom))
   )
-  (text "E" (at 254 33.02 0)
-    (effects (font (size 1.27 1.27)) (justify left bottom))
-  )
-  (text "B" (at 261.62 33.02 0)
-    (effects (font (size 1.27 1.27)) (justify left bottom))
-  )
-  (text "Transistor Die Layout (top view)" (at 243.84 27.94 0)
-    (effects (font (size 1.27 1.27)) (justify left bottom))
-  )

Commit message: Finished off the SLT-30 family of parts, started on the SLT-700 family. Changed labeling of transistors and diodes in all schematics, but have yet to update all the pdf files. This is a TODO...
Parts:
- T1: value T_DB -> DB
- T2: value T_DA -> DA
Changed lines of the file:
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@@
   (symbol (lib_id "IBM_SLT-SLD:T_DB") (at 120.65 93.98 0) (unit 1)
     (in_bom yes) (on_board yes) (fields_autoplaced)
-    (property "Reference" "T1" (id 0) (at 127 89.281 0))
-    (property "Value" "T_DB" (id 1) (at 127 91.821 0))
+    (property "Reference" "T1" (id 0) (at 124.46 93.3449 0)
+      (effects (font (size 1.27 1.27)) (justify left))
+    )
+    (property "Value" "DB" (id 1) (at 124.46 95.8849 0)
+      (effects (font (size 1.27 1.27)) (justify left))
+    )
     (property "Footprint" "Package_DFN_QFN:Diodes_DFN1006-3" (id 2) (at 120.65 93.98 0)
       (effects (font (size 1.27 1.27)) hide)
@@
   (symbol (lib_id "IBM_SLT-SLD:T_DA") (at 152.4 115.57 0) (unit 1)
     (in_bom yes) (on_board yes) (fields_autoplaced)
-    (property "Reference" "T2" (id 0) (at 158.75 110.871 0))
-    (property "Value" "T_DA" (id 1) (at 158.75 113.411 0))
+    (property "Reference" "T2" (id 0) (at 156.21 114.9349 0)
+      (effects (font (size 1.27 1.27)) (justify left))
+    )
+    (property "Value" "DA" (id 1) (at 156.21 117.4749 0)
+      (effects (font (size 1.27 1.27)) (justify left))
+    )
     (property "Footprint" "Package_DFN_QFN:Diodes_DFN1006-3" (id 2) (at 152.4 115.57 0)
       (effects (font (size 1.27 1.27)) hide)
@@
     )
     (path "/95303cff-6932-4821-b7e1-1e8ef06881c6"
-      (reference "T1") (unit 1) (value "T_DB") (footprint "Package_DFN_QFN:Diodes_DFN1006-3")
+      (reference "T1") (unit 1) (value "DB") (footprint "Package_DFN_QFN:Diodes_DFN1006-3")
     )
     (path "/aca742d5-d20c-41e7-9ac8-8b36b22cfba4"
-      (reference "T2") (unit 1) (value "T_DA") (footprint "Package_DFN_QFN:Diodes_DFN1006-3")
+      (reference "T2") (unit 1) (value "DA") (footprint "Package_DFN_QFN:Diodes_DFN1006-3")
     )
     (path "/98cf94aa-9a14-4efb-965e-894e721f61fd"
