File: SLT-30ns_AOI30-Family/361451_AI/361451_AI.kicad_sch (KiCad schematic)
At the start: 9 parts, among them T1 AAA, U1 12-Pin_SLx_Can

Commit message: Updates to 361451 AI.
Parts:
- T1: footprint (none) -> Package_TO_SOT_SMD:SOT-883
Connections:
- net 10 is gone; now on net GND: U1.10
- net GND: no longer U1.12
- new net 12: U1.12
Changed lines of the file:
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@@
-    (effects (font (size 1.27 1.27)) (justify left bottom))
-  )
-  (label "12" (at 149.86 118.11 0)
     (effects (font (size 1.27 1.27)) (justify left bottom))
   )
@@
   (label "1" (at 118.11 118.11 180)
     (effects (font (size 1.27 1.27)) (justify right bottom))
+  )
+  (label "10" (at 149.86 118.11 0)
+    (effects (font (size 1.27 1.27)) (justify left bottom))
   )
   (label "12" (at 234.95 144.78 270)
@@
       (effects (font (size 1.27 1.27)) (justify left))
     )
-    (property "Footprint" "" (id 2) (at 149.86 93.98 0)
+    (property "Footprint" "Package_TO_SOT_SMD:SOT-883" (id 2) (at 149.86 93.98 0)
       (effects (font (size 1.27 1.27)) hide)
     )
@@
     )
     (path "/5c986000-fc83-4495-a50f-9f4b94e485bc"
-      (reference "T1") (unit 1) (value "AAA") (footprint "")
+      (reference "T1") (unit 1) (value "AAA") (footprint "Package_TO_SOT_SMD:SOT-883")
     )
     (path "/75e072b9-86c1-407b-a1c4-16b7a7044004"
