File: SLT-30ns_AOI30-Family/361427_TLR2/361427_TLR2.kicad_sch (KiCad schematic)
At the start: 8 parts, among them T1 IBM_Transistor, T2 IBM_Transistor, T3 IBM_Transistor, U1 12-Pin_SLx_Can

Commit message: Finished off the SLT-30 family of parts, started on the SLT-700 family. Changed labeling of transistors and diodes in all schematics, but have yet to update all the pdf files. This is a TODO...
Parts:
- T1: value IBM_Transistor -> CC
- T2, T3: value IBM_Transistor -> ABA
Changed lines of the file:
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@@
       (effects (font (size 1.27 1.27)) (justify left))
     )
-    (property "Value" "IBM_Transistor" (id 1) (at 161.29 118.7449 0)
+    (property "Value" "ABA" (id 1) (at 161.29 118.7449 0)
       (effects (font (size 1.27 1.27)) (justify left))
     )
@@
     (in_bom yes) (on_board yes) (fields_autoplaced)
     (property "Reference" "T2" (id 0) (at 99.695 87.63 90))
-    (property "Value" "IBM_Transistor" (id 1) (at 99.695 90.17 90))
+    (property "Value" "ABA" (id 1) (at 99.695 90.17 90))
     (property "Footprint" "" (id 2) (at 100.33 82.55 0)
       (effects (font (size 1.27 1.27)) hide)
@@
       (effects (font (size 1.27 1.27)) (justify left))
     )
-    (property "Value" "IBM_Transistor" (id 1) (at 135.89 84.4549 0)
+    (property "Value" "CC" (id 1) (at 135.89 84.4549 0)
       (effects (font (size 1.27 1.27)) (justify left))
     )
@@
     )
     (path "/7b5b5180-1101-4ee8-816f-2ee7fdf5519c"
-      (reference "T1") (unit 1) (value "IBM_Transistor") (footprint "")
+      (reference "T1") (unit 1) (value "CC") (footprint "")
     )
     (path "/3aa6e313-7972-4b5e-a4c8-3414c36a4b92"
-      (reference "T2") (unit 1) (value "IBM_Transistor") (footprint "")
+      (reference "T2") (unit 1) (value "ABA") (footprint "")
     )
     (path "/328beb90-f791-4a9b-9895-c45ba1d55668"
-      (reference "T3") (unit 1) (value "IBM_Transistor") (footprint "")
+      (reference "T3") (unit 1) (value "ABA") (footprint "")
     )
     (path "/75e072b9-86c1-407b-a1c4-16b7a7044004"

Commit message: Update schematic pdfs
Other:
- note added: "361427"
Changed lines of the file:
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@@
     (effects (font (size 1.27 1.27)) (justify left bottom))
+  )
+  (text "361427" (at 107.95 101.6 0)
+    (effects (font (size 2.54 2.54)) (justify left bottom))
   )
   (label "9" (at 248.92 137.16 0)
