File: SLT-30ns_AOI30-Family/361454_DCI/361454_DCI.kicad_sch (KiCad schematic)
At the start: 7 parts, among them T1 ABB, T2 ABB, U1 12-Pin_SLx_Can

Commit message: Update schematic pdfs
Other:
- note added: "361454"
Changed lines of the file:
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@@
     (stroke (width 0) (type default) (color 0 0 0 0))
+  )
+  (text "361454" (at 109.22 76.2 0)
+    (effects (font (size 2.54 2.54)) (justify left bottom))
   )
   (label "8" (at 154.94 87.63 0)
