File: SLT-30ns_AOI30-Family/361477_XOR/361477_XOR.kicad_sch (KiCad schematic)
At the start: 8 parts, among them T1 AAB, T2 AAB, T3 ABA, U1 12-Pin_SLx_Can

Commit message: Update schematic pdfs
Other:
- note added: "361477"
Changed lines of the file:
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@@
     (stroke (width 0) (type default) (color 0 0 0 0))
+  )
+  (text "361477" (at 109.22 91.44 0)
+    (effects (font (size 2.54 2.54)) (justify left bottom))
   )
   (label "8" (at 148.59 80.645 0)
