File: SLT-700ns_AOI700-Family/361493_AI_AOI/361493_AI_AOI.kicad_sch (KiCad schematic)
At the start: 11 parts, among them T1 CB, U1 12-Pin_SLx_Can

Commit message: Add can P/N to schematics for SLT-700
Other:
- note added: "361493"
Changed lines of the file:
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@@
     (effects (font (size 1.27 1.27)) (justify left bottom))
+  )
+  (text "361493" (at 129.54 80.01 0)
+    (effects (font (size 2.54 2.54)) (justify left bottom))
   )
   (label "8" (at 170.18 63.5 0)
