File: SLT-700ns_AOI700-Family/361496_AOPX-1/361496_AOPX-1.kicad_sch (KiCad schematic)
At the start: 11 parts, among them U1 12-Pin_SLx_Can

Commit message: Add can P/N to schematics for SLT-700
Other:
- note added: "361496"
Changed lines of the file:
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@@
     (stroke (width 0) (type default) (color 0 0 0 0))
+  )
+  (text "361496" (at 111.76 66.04 0)
+    (effects (font (size 2.54 2.54)) (justify left bottom))
   )
   (text "All Diodes \"C\"" (at 111.76 133.35 0)
