File: SLT-700ns_AOI700-Family/361497_FTX/361497_FTX.kicad_sch (KiCad schematic)
At the start: 5 parts, among them T1 CA, T2 CA, T3 CA, T4 CA, U1 12-Pin_SLx_Can

Commit message: Add can P/N to schematics for SLT-700
Other:
- note added: "361497"
Changed lines of the file:
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@@
     (stroke (width 0) (type default) (color 0 0 0 0))
+  )
+  (text "361497" (at 119.38 96.52 0)
+    (effects (font (size 2.54 2.54)) (justify left bottom))
   )
   (text "All Transistors CA" (at 118.11 101.6 0)
